Commit message: Add WPG-300/120 gripper XACRO with single slider and urdf with mimic tag

File: wpg_300_120_description/urdf/wpg_300-120_meshed.urdf (robot description, URDF)
Before this commit: robot wsg_300_120, 3 links, 2 joints
Joints:
- joint right_finger_joint: mimic (none) -> joint=left_finger_joint multiplier=-1.0
